File: Eagle/IR_Bridge/schematic.brd (EAGLE design)
At the start: 49.8 x 33.2 mm, 21 parts, among them T1 2N3904, T2 2N3904, T3 2N3904, T4 2N3904, T5 2N3904, T6 2N3904, T7 2N3904

Commit message: Fix some issues on the PCB
Routing:
- net N$14: track 12.9 -> 11.9 mm
- net N$5: track 20.3 -> 19.5 mm
- net N$2: track 69.0 -> 69.5 mm
Other:
- board size 49.8 x 33.2 mm -> 50.5 x 33.2 mm
