File: Eagle/IR_Bridge/schematic.brd (EAGLE design)
At the start: 50.5 x 33.2 mm, 21 parts, among them T1 2N3904, T2 2N3904, T3 2N3904, T4 2N3904, T5 2N3904, T6 2N3904, T7 2N3904

Commit message: Schematic
Parts:
- T8: value (none) -> S8550
Changed lines of the file:
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@@
 </layers>
 <board>
+<fusionsync huburn="a.cGVyc29uYWw6dWUyZGM1OTBk" projecturn="a.cGVyc29uYWw6dWUyZGM1OTBkIzIwMTgwNDI1MTI5MjgwNjA2" f3durn="urn:adsk.wipprod:dm.lineage:OR9yDX8XTouPUYaGo1qsXA" pcbguid="cd10469c-ef26-4932-9ccc-706a7428e665" lastpulledtime="" lastsyncedchangeguid="93b634f3-2129-6691-470e-da2e81fbaf6c"/>
 <plain>
 <wire x1="-22.606" y1="-16.51" x2="27.92" y2="-16.51" width="0" layer="20"/>
@@
 <attribute name="VALUE" x="-14.66845" y="-12.255534375" size="1.27" layer="27" ratio="10"/>
 </element>
-<element name="NODEMCU" library="ESP12E_DEVKIT" package="ESP12E_DEVKIT" value="ESP12E_DEVKIT" x="1.778" y="-1.524" rot="MR90">
+<element name="NODEMCU" library="ESP12E_DEVKIT" library_urn="urn:adsk.eagle:library:2822280" package="ESP12E_DEVKIT" package3d_urn="urn:adsk.eagle:package:2822283/2" value="ESP12E_DEVKIT" x="1.778" y="-1.524" rot="MR90">
 <attribute name="MF" value="" x="1.778" y="-1.524" size="1.778" layer="28" rot="MR90" display="off"/>
 <attribute name="MPN" value="" x="1.778" y="-1.524" size="1.778" layer="28" rot="MR90" display="off"/>
@@
 <attribute name="VALUE" x="6.857996875" y="-3.6322" size="0.6096" layer="27" font="vector" ratio="20" align="top-center"/>
 </element>
-<element name="T8" library="transistor-neu-to92" library_urn="urn:adsk.eagle:library:397" package="TO92-EBC" package3d_urn="urn:adsk.eagle:package:28763/2" value="" x="16.002" y="3.556" rot="R180"/>
+<element name="T8" library="transistor-neu-to92" library_urn="urn:adsk.eagle:library:397" package="TO92-EBC" package3d_urn="urn:adsk.eagle:package:28763/2" value="S8550" x="16.002" y="3.556" rot="R180"/>
 </elements>
 <signals>
@@
 </note>
 <note version="8.3" severity="warning">
+Since Version 8.3, EAGLE supports Fusion synchronisation.
+This feature will not be available in this version and saving
+the document will break the link to the Fusion PCB feature.
+</note>
+<note version="8.3" severity="warning">
