File: Eagle/IR_Bridge/schematic.sch (EAGLE design)
At the start: 21 parts, among them T1 2N3904, T2 2N3904, T3 2N3904, T4 2N3904, T5 2N3904, T6 2N3904, T7 2N3904

Commit message: Finish designing PCB
Parts:
- renumbered U$1 to NODEMCU, U$2 to RECEIVER
Changed lines of the file:
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@@
 </classes>
 <parts>
-<part name="U$1" library="ESP12E_DEVKIT" deviceset="ESP12E_DEVKIT" device="">
+<part name="NODEMCU" library="ESP12E_DEVKIT" deviceset="ESP12E_DEVKIT" device="">
 <attribute name="MF" value=""/>
 <attribute name="MPN" value=""/>
@@
 <part name="P+6" library="supply1" library_urn="urn:adsk.eagle:library:371" deviceset="+5V" device=""/>
 <part name="P+7" library="supply1" library_urn="urn:adsk.eagle:library:371" deviceset="+5V" device=""/>
-<part name="U$2" library="tsop" deviceset="TSOP4838" device="">
+<part name="RECEIVER" library="tsop" deviceset="TSOP4838" device="">
 <attribute name="MF" value="VISHAY/TELEFUNKEN"/>
 <attribute name="MPN" value="TSOP4838"/>
@@
 </plain>
 <instances>
-<instance part="U$1" gate="G$1" x="81.28" y="50.8">
+<instance part="NODEMCU" gate="G$1" x="81.28" y="50.8">
 <attribute name="OC_NEWARK" x="81.28" y="50.8" size="1.778" layer="96" display="off"/>
 <attribute name="MF" x="81.28" y="50.8" size="1.778" layer="96" display="off"/>
@@
 <instance part="P+6" gate="1" x="129.54" y="147.32"/>
 <instance part="P+7" gate="1" x="109.22" y="101.6"/>
-<instance part="U$2" gate="G$1" x="144.78" y="48.26" rot="R180">
+<instance part="RECEIVER" gate="G$1" x="144.78" y="48.26" rot="R180">
 <attribute name="OC_NEWARK" x="144.78" y="48.26" size="1.778" layer="96" display="off"/>
 <attribute name="MF" x="144.78" y="48.26" size="1.778" layer="96" display="off"/>
@@
 <pinref part="R1" gate="G$1" pin="2"/>
 <wire x1="109.22" y1="68.58" x2="111.76" y2="68.58" width="0.1524" layer="91"/>
-<pinref part="U$1" gate="G$1" pin="D2"/>
+<pinref part="NODEMCU" gate="G$1" pin="D2"/>
 <wire x1="99.06" y1="63.5" x2="109.22" y2="63.5" width="0.1524" layer="91"/>
 <wire x1="109.22" y1="63.5" x2="109.22" y2="68.58" width="0.1524" layer="91"/>
@@
 </segment>
 <segment>
-<pinref part="U$1" gate="G$1" pin="GND@3"/>
+<pinref part="NODEMCU" gate="G$1" pin="GND@3"/>
 <wire x1="99.06" y1="35.56" x2="106.68" y2="35.56" width="0.1524" layer="91"/>
 <pinref part="GND1" gate="1" pin="GND"/>
@@
 <pinref part="T1" gate="G1" pin="E"/>
 <wire x1="129.54" y1="63.5" x2="129.54" y2="60.96" width="0.1524" layer="91"/>
-<pinref part="U$2" gate="G$1" pin="GND"/>
+<pinref part="RECEIVER" gate="G$1" pin="GND"/>
 <wire x1="129.54" y1="60.96" x2="129.54" y2="58.42" width="0.1524" layer="91"/>
 <wire x1="137.16" y1="53.34" x2="137.16" y2="60.96" width="0.1524" layer="91"/>
@@
 <net name="+5V" class="0">
 <segment>
-<pinref part="U$1" gate="G$1" pin="VIN"/>
+<pinref part="NODEMCU" gate="G$1" pin="VIN"/>
 <wire x1="63.5" y1="33.02" x2="53.34" y2="33.02" width="0.1524" layer="91"/>
 <pinref part="P+1" gate="1" pin="+5V"/>
@@
 </segment>
 <segment>
-<pinref part="U$2" gate="G$1" pin="V+"/>
+<pinref part="RECEIVER" gate="G$1" pin="V+"/>
 <pinref part="P+8" gate="1" pin="+5V"/>
 <wire x1="137.16" y1="43.18" x2="132.08" y2="43.18" width="0.1524" layer="91"/>
@@
 <net name="N$6" class="0">
 <segment>
-<pinref part="U$2" gate="G$1" pin="OUT"/>
+<pinref part="RECEIVER" gate="G$1" pin="OUT"/>
 <wire x1="137.16" y1="48.26" x2="111.76" y2="48.26" width="0.1524" layer="91"/>
 <wire x1="111.76" y1="48.26" x2="111.76" y2="66.04" width="0.1524" layer="91"/>
-<pinref part="U$1" gate="G$1" pin="D1"/>
+<pinref part="NODEMCU" gate="G$1" pin="D1"/>
 <wire x1="111.76" y1="66.04" x2="99.06" y2="66.04" width="0.1524" layer="91"/>
 </segment>

Commit message: Schematic
Parts:
- T8: value (none) -> S8550
Changed lines of the file:
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@@
 <?xml version="1.0" encoding="utf-8"?>
 <!DOCTYPE eagle SYSTEM "eagle.dtd">
-<eagle version="8.7.1">
+<eagle version="9.0.0">
 <drawing>
 <settings>
@@
 </classes>
 <parts>
-<part name="NODEMCU" library="ESP12E_DEVKIT" deviceset="ESP12E_DEVKIT" device="">
+<part name="NODEMCU" library="ESP12E_DEVKIT" library_urn="urn:adsk.eagle:library:2822280" deviceset="ESP12E_DEVKIT" device="" package3d_urn="urn:adsk.eagle:package:2822283/2">
 <attribute name="MF" value=""/>
 <attribute name="MPN" value=""/>
@@
 </part>
 <part name="P+9" library="supply1" library_urn="urn:adsk.eagle:library:371" deviceset="+5V" device=""/>
-<part name="T8" library="transistor-neu-to92" library_urn="urn:adsk.eagle:library:397" deviceset="*-PNP-" device="TO92-EBC" package3d_urn="urn:adsk.eagle:package:28763/2"/>
+<part name="T8" library="transistor-neu-to92" library_urn="urn:adsk.eagle:library:397" deviceset="*-PNP-" device="TO92-EBC" package3d_urn="urn:adsk.eagle:package:28763/2" value="S8550"/>
 </parts>
 <sheets>
